File: pcb-projects/particle-tiny1634/particle.kicad_pcb (KiCad board)
At the start: 2 copper layers, 42.5 x 43.2 mm, 32 parts, among them CON1 AVR-ISP-6, IC1 ATTINY1634-SU, P1 TXN, P2 RXN, P3 TXS, P4 RXS, P5 TRX-CH, P6 TEST1-3

Commit message: routed pluggable particle
Other:
- board text added: "V 1.1 12/2015"
Changed lines of the file:
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@@
     (area 133.909999 85.014999 176.605001 128.345001)
     (thickness 1.6)
-    (drawings 12)
+    (drawings 13)
     (tracks 361)
     (zones 0)
@@
     )
   )
+  (gr_text "V 1.1\n12/2015" (at 170.18 88.265) (layer Dwgs.User)
+    (effects (font (size 1.5 1.5) (thickness 0.3)))
+  )
   (gr_text + (at 164.465 119.38) (layer F.Cu)
