File: pcb-projects/particle-tiny1634-pluggable-module/particle-tiny1634-plugable-module.kicad_pcb (KiCad board)
At the start: 2 copper layers, 37.5 x 45.7 mm, 32 parts, among them IC1 ATTINY1634-SU, P1 INTERFACE, P2 MCU_TEST

Commit message: cleanup folders; minimal pcb changes
Parts:
- added C1: 100nF, Capacitors_SMD:C_1206_HandSoldering, F.Cu at (154.9, 93.0)
- moved R8 2.60 mm to (154.9, 89.5)
- renumbered Q-CHAIN1 to Q-EAST1
Connections:
- net /PWR/TX-CHAIN renamed /SW_PWR_TX-EAST
- net /PWR/TX-NORTH renamed /SW_PWR_TX-NORTH
- net /PWR/TX-SOUTH renamed /SW_PWR_TX-SOUTH
- net /RX-CHAIN renamed /RX-EAST
- net /SW_PWR/RX-CHAIN renamed /SW_PWR_RX-EAST
- net /SW_PWR/RX-NORTH renamed /SW_PWR_RX-NORTH
- net /SW_PWR/RX-SOUTH renamed /SW_PWR_RX-SOUTH
- net /TX-CHAIN renamed /TX-EAST
Routing:
- net GND: track 95.8 -> 108.4 mm, vias 9 -> 10
- net /RX-NORTH: track 75.6 -> 74.0 mm
- net VCC: track 141.3 -> 142.1 mm
- net /RX-SOUTH: track 29.8 -> 29.1 mm
- added copper zone on F.Cu, net GND
Other:
- outline, holes or cut-outs redrawn
- net class Default: via_dia 1.2 -> 1.4
- board text added: "01/2016"
- board text added: "RR"
- board text added: "V1.21"
- board text removed: "12"
- board text removed: "RAOUL RUBIEN"
- board text removed: "V1.2 01/2016"
